File: MCU_PCB/main_controller/main_controller.sch (KiCad schematic (older format))
At the start: 38 parts, among them J1 TB006-508-05BE, J2 TB006-508-05BE, J3 TB006-508-05BE, J4 TB006-508-05BE, J5 1715250000, Q1 Q_PMOS_GSD, SW1 SW_SPDT, U1 STM32F446ZET6

Commit message: Finished with PCB model 1
Parts:
- removed D1: D_Schottky, symbol Device:D_Schottky
- removed ESD1: USBLC6-2SC6, Package_TO_SOT_SMD:SOT-23-6, symbol Power_Protection:USBLC6-2SC6
- removed J3: TB006-508-05BE, SHDR5W100P0X508_1X5_2540X820X1000P, symbol TB006-508-05BE:TB006-508-05BE
- removed Q1: Q_PMOS_GSD, DMP3098LSS-13:SOIC127P600X175-8N, symbol Device:Q_PMOS_GSD
- removed R5, R6: 2.2k, Resistor_SMD:R_0805_2012Metric, symbol Device:R_Small
- removed USB_J1: USB_B_Micro, SamacSys_Parts:USB313530A, symbol Connector:USB_B_Micro
- added C20, C21: C_Small, Capacitor_SMD:C_0805_2012Metric, symbol Device:C_Small
- added Y1: Crystal_GND24_Small, EA1620LA12-16.000M_TR:EA1620LA1216000MTR, symbol Device:Crystal_GND24_Small
- D2: footprint (none) -> LED_SMD:LED_0805_2012Metric
- J1, J2, J4: footprint SHDR5W100P0X508_1X5_2540X820X1000P -> SamacSys_Parts:SHDR5W100P0X508_1X5_2540X820X1000P; symbol TB006-508-05BE:TB006-508-05BE -> main_controller-rescue:TB006-508-05BE-TB006-508-05BE
- J5: symbol SamacSys_Parts:1715250000 -> main_controller-rescue:1715250000-SamacSys_Parts
- L1: footprint (none) -> Inductor_SMD:L_0402_1005Metric
- SW1: footprint (none) -> spdt switch:118251376
- SWD1: footprint (none) -> Connector_PinHeader_2.54mm:PinHeader_1x06_P2.54mm_Vertical
Connections:
- net labels added: 12V, 3V3, 5V, 7.5V, 7.5V_IN, TIM3_CH2, TIM4_CH3, TIM4_CH4, WIFI_EN, WIFI_nRST
- net labels removed: +12V, +5V, 3.3V_reg_in, GPIO1, GPIO2, GPIO3, I2C1_SCL, I2C1_SDA, USART2_RX, USART2_TX, USART6_RX, USART6_TX, USB_CONN_D+, USB_CONN_D-, USB_D+, USB_D-
- wire segments 177 -> 167
- no-connect marks 88 -> 81
Other:
- note added: "Filters the 7.5V"
- note added: "connect pin 39 to C7 (decoup cap)\n"
- note removed: "This is a circuit for reverse polarity protection for the Circuit"
- note removed: "USB Micro Power + ESD Protection"
- moved on the sheet: C13, C5, D2, FB1, R4
