File: MCU_PCB/main_controller/main_controller.sch (KiCad schematic (older format))
At the start: 55 parts, among them J1 TB006-508-05BE, J2 TB006-508-05BE, J4 TB006-508-05BE, J5 1715250000, SW1 SW_SPDT, SW4 KEY_FLASH, U1 STM32F446ZET6, Y1 Crystal_GND24_Small

Commit message: Finishing up small airwires
Parts:
- C1, C10, C11, C12, C13, C14, C15, C16, C17, C2, C20, C21, C3, C4, C5, C6, C7, C8, C9: symbol Device:C_Small -> main_controller-rescue:C_Small-Device
- C30: symbol Device:CP1 -> main_controller-rescue:CP1-Device
- C?: symbol Device:C -> main_controller-rescue:C-Device
- D1, D2, D5, D6, D7, D8: symbol Device:LED -> main_controller-rescue:LED-Device
- D9: symbol Device:D -> main_controller-rescue:D-Device
- F1: symbol Device:Polyfuse_Small -> main_controller-rescue:Polyfuse_Small-Device
- FB1: symbol Device:Ferrite_Bead_Small -> main_controller-rescue:Ferrite_Bead_Small-Device
- L1: symbol Device:L_Small -> main_controller-rescue:L_Small-Device
- R1, R26, R3, R4: symbol Device:R_Small -> main_controller-rescue:R_Small-Device
- R15, R16, R18, R2, R21, R22, R23, R24, R25, R5, R6: symbol Device:R -> main_controller-rescue:R-Device
- SW1: symbol Switch:SW_SPDT -> main_controller-rescue:SW_SPDT-Switch
- SW4: symbol Switch:SW_Push -> main_controller-rescue:SW_Push-Switch
- SWD1: symbol Connector:Conn_01x06_Female -> main_controller-rescue:Conn_01x06_Female-Connector
- U1: symbol MCU_ST_STM32F4:STM32F446ZETx -> main_controller-rescue:STM32F446ZETx-MCU_ST_STM32F4
- Y1: symbol Device:Crystal_GND24_Small -> main_controller-rescue:Crystal_GND24_Small-Device
