File: MCU_PCB/main_controller/_autosave-file616037F9.sch (KiCad schematic (older format))
At the start: 30 parts, among them IC5 esp-12f, J8 USB_B_Micro, Q2 S8050, Q3 S8050, SW2 KEY_USER, SW3 KEY_FLASH, U3 CH340G, U4 R-78E5.0-0.5, U5 ISE0512A-H, X1 ECS-2520MV-xxx-xx

Commit message: finished drc check
Parts:
- removed U5: ISE0512A-H, 5to3.3:ISE0512A-H, symbol 5to3.3:ISE0512A-H
- added J3: VX7803-500, NEW5TO3V3:VX7803-500, symbol 5to3v3:VX7803-500
Changed lines of the file:
@@
 	1    0    0    -1
 $EndComp
-$Comp
-L 5to3.3:ISE0512A-H U?
-U 1 1 615F56D6
-P 3100 3200
-AR Path="/61651051/615F56D6" Ref="U?"  Part="1"
-AR Path="/616037FA/615F56D6" Ref="U5"  Part="1"
-F 0 "U5" H 3900 3693 60  0000 C CNN
-F 1 "ISE0512A-H" H 3900 3587 60  0000 C CNN
-F 2 "5to3.3:ISE0512A-H" H 3900 3481 60  0000 C CNN
-F 3 "" H 3100 3200 60  0000 C CNN
-	1    3100 3200
-	1    0    0    -1
-$EndComp
-Text GLabel 3100 3200 0    50   Input ~ 0
-5V
-Text GLabel 4700 3300 2    50   Input ~ 0
-3V3
-Text GLabel 4700 3400 2    50   Input ~ 0
-GND
-Text GLabel 3100 3300 0    50   Input ~ 0
-GND
 Text GLabel 5550 3850 0    50   Input ~ 0
 7.5V
@@
 	1    0    0    -1
 $EndComp
+$Comp
+L 5to3v3:VX7803-500 J3
+U 1 1 6198DC88
+P 3850 3500
+F 0 "J3" H 4378 3453 60  0000 L CNN
+F 1 "VX7803-500" H 4378 3347 60  0000 L CNN
+F 2 "NEW5TO3V3:VX7803-500" H 4250 3340 60  0001 C CNN
+F 3 "" H 3850 3500 60  0000 C CNN
+	1    3850 3500
+	1    0    0    -1
+$EndComp
+Text GLabel 3850 3500 0    39   Input ~ 0
+5V
+Text GLabel 3850 3700 0    39   Input ~ 0
+3V3
+Text GLabel 3850 3600 0    39   Input ~ 0
+GND
 $EndSCHEMATC

Commit message: Adding footprints/schematics locally
Parts:
- removed J8: USB_B_Micro, usbtomicro:J_SMD_2174507-2-5_7.8_5_2.71, symbol Connector:USB_B_Micro
- added J6: 2174507-2, microusb_b:2174507-2, symbol microusb_b:2174507-2
Connections:
- wire segments 68 -> 65
Changed lines of the file:
@@
 Text Label 4950 6450 0    50   ~ 0
 5V
-$Comp
-L Connector:USB_B_Micro J8
-U 1 1 6157029C
-P 8600 5700
-F 0 "J8" H 8370 5597 50  0000 R CNN
-F 1 "USB_B_Micro" H 8370 5688 50  0000 R CNN
-F 2 "usbtomicro:J_SMD_2174507-2-5_7.8_5_2.71" H 8750 5650 50  0001 C CNN
-F 3 "~" H 8750 5650 50  0001 C CNN
-	1    8600 5700
-	-1   0    0    1
-$EndComp
-Wire Wire Line
-	8300 5900 8200 5900
-Wire Wire Line
-	8200 5900 8200 6050
-NoConn ~ 8300 5500
 Text Label 10950 6250 0    50   ~ 0
 GND
@@
 GND
 Text Label 5400 6950 3    50   ~ 0
-GND
-Text Label 8600 5300 1    50   ~ 0
 GND
 $Comp
@@
 	1    0    0    -1
 $EndComp
-Text Label 8200 6400 3    50   ~ 0
-5V
 $Comp
 L main_controller-rescue:USBLC6-2SC6-Power_Protection ESD?
@@
 Text GLabel 7450 5450 2    25   Input ~ 0
 USB_D+
-Text GLabel 8300 5700 0    25   Input ~ 0
-USB_CONN_D+
-Text GLabel 8300 5600 0    25   Input ~ 0
-USB_CONN_D-
 Text GLabel 5900 5650 2    25   Input ~ 0
 USB_D-
 Text GLabel 5900 5750 2    25   Input ~ 0
 USB_D+
-Wire Wire Line
-	8200 6350 8200 6400
-$Comp
-L Device:D_Schottky D3
-U 1 1 61572E44
-P 8200 6200
-F 0 "D3" V 8246 6121 50  0000 R CNN
-F 1 "D_Schottky" V 8155 6121 50  0000 R CNN
-F 2 "Diode 4007:1N4007G-T" H 8150 5650 50  0000 C CNN
-F 3 "~" H 8200 6200 50  0001 C CNN
-	1    8200 6200
-	0    -1   -1   0
-$EndComp
 Text Label 10050 1450 0    50   ~ 0
 XI
@@
 Text GLabel 3850 3600 0    39   Input ~ 0
 GND
+$Comp
+L microusb_b:2174507-2 J6
+U 1 1 6199C811
+P 9750 5350
+F 0 "J6" H 10478 4903 60  0000 L CNN
+F 1 "2174507-2" H 10478 4797 60  0000 L CNN
+F 2 "microusb_b:2174507-2" H 10150 5090 60  0001 C CNN
+F 3 "" H 9750 5350 60  0000 C CNN
+	1    9750 5350
+	1    0    0    -1
+$EndComp
+$Comp
+L Device:D_Schottky D3
+U 1 1 619A2A55
+P 9600 5350
+F 0 "D3" V 9646 5271 50  0000 R CNN
+F 1 "D_Schottky" V 9555 5271 50  0000 R CNN
+F 2 "Diode 4007:1N4007G-T" H 9550 4800 50  0000 C CNN
+F 3 "~" H 9600 5350 50  0001 C CNN
+	1    9600 5350
+	1    0    0    -1
+$EndComp
+Text GLabel 9450 5350 0    39   Input ~ 0
+5V
+Text GLabel 9750 5550 0    25   Input ~ 0
+USB_CONN_D+
+Text GLabel 9750 5450 0    25   Input ~ 0
+USB_CONN_D-
+NoConn ~ 9750 5650
+Text GLabel 9750 5750 0    39   Input ~ 0
+GND
 $EndSCHEMATC

Commit message: Working more on footprint adjustments
Parts:
- D3: footprint Diode 4007:1N4007G-T -> walle_library:1N4007G-T
- IC5: footprint esp12f -> walle_library:esp12f
- J3: footprint NEW5TO3V3:VX7803-500 -> walle_library:VX7803-500
- J6: footprint microusb_b:2174507-2 -> walle_library:2174507-2
- SW2, SW3: footprint pushbutton:SW_147873-2 -> walle_library:SW_147873-2
- U4: footprint DC 7.5 to 5:R-78E5.0-0.5 -> walle_library:R-78E5.0-0.5
Changed lines of the file:
@@
 F 0 "IC5" H 6050 1115 50  0000 C CNN
 F 1 "esp-12f" H 6050 1024 50  0000 C CNN
-F 2 "esp12f" H 6550 950 50  0001 L CNN
+F 2 "walle_library:esp12f" H 6550 950 50  0001 L CNN
 F 3 "https://docs.ai-thinker.com/_media/esp8266/docs/esp-12f_product_specification_en.pdf" H 6550 850 50  0001 L CNN
 F 4 "ESP-12F ESP8266 Wifi Wireless IoT Board Module , package 1 x ESP8266 Adapter Plate  1pcs" H 6550 750 50  0001 L CNN "Description"
@@
 F 0 "SW2" V 9054 4848 50  0000 L CNN
 F 1 "KEY_USER" V 9145 4848 50  0000 L CNN
-F 2 "pushbutton:SW_147873-2" H 9100 4900 50  0000 C CNN
+F 2 "walle_library:SW_147873-2" H 9100 4900 50  0000 C CNN
 F 3 "~" H 9100 4900 50  0001 C CNN
 	1    9100 4700
@@
 F 0 "SW3" V 10454 4798 50  0000 L CNN
 F 1 "KEY_FLASH" V 10545 4798 50  0000 L CNN
-F 2 "pushbutton:SW_147873-2" H 10500 4850 50  0000 C CNN
+F 2 "walle_library:SW_147873-2" H 10500 4850 50  0000 C CNN
 F 3 "~" H 10500 4850 50  0001 C CNN
 	1    10500 4650
@@
 F 0 "U4" H 6350 4237 60  0000 C CNN
 F 1 "R-78E5.0-0.5" H 6350 4131 60  0000 C CNN
-F 2 "DC 7.5 to 5:R-78E5.0-0.5" H 6350 4090 60  0001 C CNN
+F 2 "walle_library:R-78E5.0-0.5" H 6350 4090 60  0001 C CNN
 F 3 "" H 5550 3850 60  0000 C CNN
 	1    5550 3850
@@
 F 0 "J3" H 4378 3453 60  0000 L CNN
 F 1 "VX7803-500" H 4378 3347 60  0000 L CNN
-F 2 "NEW5TO3V3:VX7803-500" H 4250 3340 60  0001 C CNN
+F 2 "walle_library:VX7803-500" H 4250 3340 60  0001 C CNN
 F 3 "" H 3850 3500 60  0000 C CNN
 	1    3850 3500
@@
 F 0 "J6" H 10478 4903 60  0000 L CNN
 F 1 "2174507-2" H 10478 4797 60  0000 L CNN
-F 2 "microusb_b:2174507-2" H 10150 5090 60  0001 C CNN
+F 2 "walle_library:2174507-2" H 10150 5090 60  0001 C CNN
 F 3 "" H 9750 5350 60  0000 C CNN
 	1    9750 5350
@@
 F 0 "D3" V 9646 5271 50  0000 R CNN
 F 1 "D_Schottky" V 9555 5271 50  0000 R CNN
-F 2 "Diode 4007:1N4007G-T" H 9550 4800 50  0000 C CNN
+F 2 "walle_library:1N4007G-T" H 9550 4800 50  0000 C CNN
 F 3 "~" H 9600 5350 50  0001 C CNN
 	1    9600 5350

Commit message: Archived main board
Connections:
- net labels removed: ADC
- wire segments 65 -> 64
Other:
- moved on the sheet: C23, C24, ESD1, Q2, Q3, R11, R12, R13, R14, U3
