File: MCU_PCB/main_controller/_autosave-main_controller.kicad_pcb (KiCad board)
At the start: 2 copper layers, 94.8 x 89.5 mm, 82 parts, among them IC5 esp-12f, J1 TB006-508-05BE, J2 TB006-508-05BE, J3 VX7803-500, J4 TB006-508-05BE, J5 1715250000, J6 2174507-2, Q2 S8050, Q3 S8050, SW1 SW_SPDT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

Commit message: Working more on footprint adjustments
Changed lines of the file:
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@@
     (thickness 1.6)
     (drawings 14)
-    (tracks 639)
+    (tracks 640)
     (zones 0)
     (modules 82)
@@
   (segment (start 116.7 36.35) (end 116.825 36.225) (width 0.4064) (layer F.Cu) (net 150))
   (segment (start 111.555 36.35) (end 116.7 36.35) (width 0.4064) (layer F.Cu) (net 150))
-  (segment (start 161.375 35.11) (end 160.64 34.375) (width 0.25) (layer F.Cu) (net 165))
-  (segment (start 161.375 59.6375) (end 161.375 35.11) (width 0.25) (layer F.Cu) (net 165))
+  (segment (start 160.64 34.375) (end 160.64 37.34) (width 0.25) (layer F.Cu) (net 165))
+  (segment (start 160.64 37.34) (end 161.375 38.075) (width 0.25) (layer F.Cu) (net 165))
+  (segment (start 161.375 59.6375) (end 161.375 38.075) (width 0.25) (layer F.Cu) (net 165))
   (segment (start 148.525 53.7875) (end 148.525 51.3625) (width 0.25) (layer F.Cu) (net 167))
   (segment (start 154.10001 62.00001) (end 149.57501 62.00001) (width 0.25) (layer F.Cu) (net 168))

Commit message: Archived main board
Parts:
- removed G***: LOGO, walle_library:walle3
- removed the REF** at (188.5, 44.1)
- removed the REF** at (139.6, 44.0)
- removed the REF** at (105.7, 112.8)
- removed the REF** at (193.2, 112.3)
- added REF**: MountingHole_2.2mm_M2, MountingHole:MountingHole_2.2mm_M2, F.Cu at (143.0, 32.7)
- added REF**: MountingHole_2.2mm_M2, MountingHole:MountingHole_2.2mm_M2, F.Cu at (192.0, 111.8)
- added REF**: MountingHole_2.2mm_M2, MountingHole:MountingHole_2.2mm_M2, F.Cu at (105.9, 113.2)
- D3: footprint Diode 4007:1N4007G-T -> walle_library:1N4007G-T
- IC5: footprint esp12f -> walle_library:esp12f
- J3: footprint NEW5TO3V3:VX7803-500 -> walle_library:VX7803-500
- J6: footprint microusb_b:2174507-2 -> walle_library:2174507-2
- SW1: footprint spdt switch:118251376 -> walle_library:118251376
- SW2, SW3: footprint pushbutton:SW_147873-2 -> walle_library:SW_147873-2
- U4: footprint DC 7.5 to 5:R-78E5.0-0.5 -> walle_library:R-78E5.0-0.5
- Y1: footprint EA1620LA12-16.000M_TR:EA1620LA1216000MTR -> walle_library:EA1620LA1216000MTR
- moved R18 8.98 mm to (138.6, 45.5)
- moved R21 8.98 mm to (141.9, 45.4)
Routing:
- net 12V: track 39.8 -> 45.7 mm
- net ADC3_IN5: track 41.1 -> 39.0 mm
