File: MCU_PCB/main_controller/_autosave-main_controller.sch (KiCad schematic (older format))
At the start: 44 parts, among them J1 TB006-508-05BE, J2 TB006-508-05BE, J4 TB006-508-05BE, J5 1715250000, SW1 SW_SPDT, U1 STM32F446ZET6, Y1 Crystal_GND24_Small

Commit message: finished drc check
Parts:
- added R18: 10k, Resistor_SMD:R_0805_2012Metric, symbol Device:R
- added R21: 2k, Resistor_SMD:R_0805_2012Metric, symbol Device:R
- D1: footprint (none) -> LED_SMD:LED_0805_2012Metric
Connections:
- net 12V: now also R18.1
- net ADC3_IN5: now also R18.2, R21.1
- net GND: now also R21.2
Changed lines of the file:
@@
 F 0 "D1" H 4143 545 50  0000 C CNN
 F 1 "LED" H 4143 636 50  0000 C CNN
-F 2 "" H 4150 800 50  0001 C CNN
+F 2 "LED_SMD:LED_0805_2012Metric" H 4150 800 50  0001 C CNN
 F 3 "~" H 4150 800 50  0001 C CNN
 	1    4150 800
@@
 	0    -1   -1   0
 $EndComp
+$Comp
+L Device:R R18
+U 1 1 6193B4E2
+P 1300 4900
+F 0 "R18" H 1370 4946 50  0000 L CNN
+F 1 "10k" H 1370 4855 50  0000 L CNN
+F 2 "Resistor_SMD:R_0805_2012Metric" V 1230 4900 50  0001 C CNN
+F 3 "~" H 1300 4900 50  0001 C CNN
+	1    1300 4900
+	1    0    0    -1
+$EndComp
+$Comp
+L Device:R R21
+U 1 1 6193B99E
+P 1300 5400
+F 0 "R21" H 1370 5446 50  0000 L CNN
+F 1 "2k" H 1370 5355 50  0000 L CNN
+F 2 "Resistor_SMD:R_0805_2012Metric" V 1230 5400 50  0001 C CNN
+F 3 "~" H 1300 5400 50  0001 C CNN
+	1    1300 5400
+	1    0    0    -1
+$EndComp
+Wire Wire Line
+	1300 5050 1300 5150
+Wire Wire Line
+	1300 4750 1300 4600
+$Comp
+L power:GND #PWR01
+U 1 1 6195F3F7
+P 1300 5550
+F 0 "#PWR01" H 1300 5300 50  0001 C CNN
+F 1 "GND" H 1305 5377 50  0000 C CNN
+F 2 "" H 1300 5550 50  0001 C CNN
+F 3 "" H 1300 5550 50  0001 C CNN
+	1    1300 5550
+	1    0    0    -1
+$EndComp
+Text GLabel 1300 4600 1    50   Input ~ 0
+12V
+Wire Wire Line
+	1300 5150 1550 5150
+Connection ~ 1300 5150
+Wire Wire Line
+	1300 5150 1300 5250
+Text GLabel 1550 5150 2    25   Input ~ 0
+ADC3_IN5
 $EndSCHEMATC

Commit message: Adding footprints/schematics locally
Parts:
- added R22: 0, Resistor_SMD:R_0805_2012Metric, symbol Device:R
Connections:
- net 3.3V_regulator is gone; now on net +3V3: SWD1.1 (Pin_1)
- net GND: now also R22.2; no longer C14.2, C15.2, C5.2
- new net AGND: C14.2, C15.2, C5.2, R22.1
Changed lines of the file:
@@
 	10050 1400 10050 1250
-$Comp
-L power:GND #PWR0111
-U 1 1 6160194E
-P 10450 1400
-F 0 "#PWR0111" H 10450 1150 50  0001 C CNN
-F 1 "GND" H 10455 1227 50  0000 C CNN
-F 2 "" H 10450 1400 50  0001 C CNN
-F 3 "" H 10450 1400 50  0001 C CNN
-	1    10450 1400
-	1    0    0    -1
-$EndComp
-Connection ~ 10450 1400
 $Comp
 L power:+3.3VA #PWR0112
@@
 	4050 7100 3850 7100
 Text GLabel 3850 6600 0    25   Input ~ 0
-3.3V_regulator
+3V3
 Text GLabel 3850 6700 0    25   Input ~ 0
 SWCLK
@@
 	0    -1   -1   0
 $EndComp
-$Comp
-L power:GND #PWR0117
-U 1 1 6191ED8D
-P 9650 5350
-F 0 "#PWR0117" H 9650 5100 50  0001 C CNN
-F 1 "GND" H 9655 5177 50  0000 C CNN
-F 2 "" H 9650 5350 50  0001 C CNN
-F 3 "" H 9650 5350 50  0001 C CNN
-	1    9650 5350
-	0    -1   -1   0
-$EndComp
 Text Notes 9600 3000 0    50   ~ 0
 connect pin 39 to C7 (decoup cap)\n
@@
 Text GLabel 1550 5150 2    25   Input ~ 0
 ADC3_IN5
+Text Label 9650 5350 0    39   ~ 0
+AGND
+Text Label 10450 1400 0    39   ~ 0
+AGND
+$Comp
+L Device:R R22
+U 1 1 619EA822
+P 9200 1300
+F 0 "R22" H 9270 1346 50  0000 L CNN
+F 1 "0" H 9270 1255 50  0000 L CNN
+F 2 "Resistor_SMD:R_0805_2012Metric" V 9130 1300 50  0001 C CNN
+F 3 "~" H 9200 1300 50  0001 C CNN
+	1    9200 1300
+	1    0    0    -1
+$EndComp
+Text Label 9200 1150 0    39   ~ 0
+AGND
+Text Label 9200 1450 0    39   ~ 0
+GND
 $EndSCHEMATC

Commit message: Working more on footprint adjustments
Parts:
- SW1: footprint spdt switch:118251376 -> walle_library:118251376
- Y1: footprint EA1620LA12-16.000M_TR:EA1620LA1216000MTR -> walle_library:EA1620LA1216000MTR
Changed lines of the file:
@@
 F 0 "SW1" H 7400 1235 50  0000 C CNN
 F 1 "SW_SPDT" H 7400 1144 50  0000 C CNN
-F 2 "spdt switch:118251376" H 7400 950 50  0001 C CNN
+F 2 "walle_library:118251376" H 7400 950 50  0001 C CNN
 F 3 "~" H 7400 950 50  0001 C CNN
 	1    7400 950
@@
 F 0 "Y1" H 1094 3350 50  0000 L CNN
 F 1 "Crystal_GND24_Small" H 1094 3305 50  0001 L CNN
-F 2 "EA1620LA12-16.000M_TR:EA1620LA1216000MTR" H 950 3350 50  0001 C CNN
+F 2 "walle_library:EA1620LA1216000MTR" H 950 3350 50  0001 C CNN
 F 3 "~" H 950 3350 50  0001 C CNN
 	1    950  3350

Commit message: Archived main board
Other:
- moved on the sheet: C20, C21, C5, D1, D5, D6, D7, D8, R15, R16, R18, R2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
