File: MCU_PCB/main_controller/main_controller.kicad_pcb (KiCad board)
At the start: 2 copper layers, 94.8 x 89.5 mm, 86 parts, among them IC5 esp-12f, J1 TB006-508-05BE, J2 TB006-508-05BE, J3 VX7803-500, J4 TB006-508-05BE, J5 1715250000, J6 2174507-2, Q2 S8050, Q3 S8050, SW1 SW_SPDT, SW2 KEY_USER, SW3 KEY_FLASH, U1 STM32F446ZET6, U3 CH340G, X1 ECS-2520MV-xxx-xx, Y1 Crystal_GND24_Small

Commit message: Almost approved
Parts:
- removed X1: ECS-2520MV-xxx-xx, Oscillator:Oscillator_SMD_ECS_2520MV-xxx-xx-4Pin_2.5x2.0mm
- added C30: 100uF, walle_library:CAP_EEEHA0J101WR, F.Cu at (119.2, 31.8)
- added D9: D, Diode_SMD:D_0805_2012Metric, B.Cu at (161.8, 67.4)
- added G***: LOGO, walle_library:walle, F.Cu at (172.1, 97.2)
- added R23: R, Resistor_SMD:R_0805_2012Metric, F.Cu at (194.8, 54.2)
- added R24: 10, Resistor_SMD:R_0805_2012Metric, F.Cu at (183.2, 97.0)
- added R25: 10, Resistor_SMD:R_0805_2012Metric, F.Cu at (183.9, 92.2)
- added R26: 22, Resistor_SMD:R_0805_2012Metric, F.Cu at (187.3, 58.2)
- added SW4: KEY_FLASH, walle_library:SW_147873-2, F.Cu at (193.7, 45.5)
- added Y2: ABM3B-12.000MHZ, walle_library:ABM3B-12.000MHZ, F.Cu at (115.8, 83.6)
- C18: footprint EEEHA0J101WR:CAP_EEEHA0J101WR -> walle_library:CAP_EEEHA0J101WR
- C22: moved to B.Cu
- TP1, TP2: footprint TestPoint:TestPoint_Loop_D2.50mm_Drill1.0mm -> walle_library:KEYSTONE_5000
- moved C25 3.37 mm to (119.7, 87.8)
- moved R18 3.15 mm to (141.7, 45.6)
- moved R21 3.15 mm to (145.0, 45.5)
- moved PS1 2.72 mm to (129.4, 37.6)
- moved C22 2.40 mm to (137.0, 43.0)
- moved C26 0.91 mm to (112.3, 83.9)
- moved C29 0.84 mm to (132.8, 33.8)
- moved C2 0.78 mm to (163.7, 63.1)
- moved H3 0.71 mm to (143.5, 34.3)
- moved FB1 0.66 mm to (119.1, 42.1)
- moved C28 0.15 mm to (128.1, 42.9), turned to 0 degrees
- moved TP1 0.06 mm to (104.7, 103.1), turned to 0 degrees
Connections:
- C19 pad 2: WIFI_nRST -> 3V3
- D4 pad 1: Net-(D4-Pad1) -> /WiFi + MCU/GPIO16
- D4 pad 2: /WiFi + MCU/GPIO16 -> Net-(D4-Pad2)
- ESD1 pad 5: (no net) -> +5V
- IC5 pad 1: WIFI_nRST -> 3V3
- IC5 pad 10: (no net) -> Net-(IC5-Pad10)
- IC5 pad 11: (no net) -> Net-(IC5-Pad11)
- IC5 pad 12: (no net) -> Net-(IC5-Pad12)
- IC5 pad 13: (no net) -> Net-(IC5-Pad13)
- IC5 pad 14: (no net) -> Net-(IC5-Pad14)
- IC5 pad 16: (no net) -> Net-(IC5-Pad16)
- IC5 pad 17: (no net) -> Net-(IC5-Pad17)
- IC5 pad 19: (no net) -> Net-(IC5-Pad19)
- IC5 pad 2: (no net) -> Net-(IC5-Pad2)
- IC5 pad 20: (no net) -> Net-(IC5-Pad20)
- IC5 pad 5: (no net) -> Net-(IC5-Pad5)
- IC5 pad 6: (no net) -> Net-(IC5-Pad6)
- IC5 pad 7: (no net) -> Net-(IC5-Pad7)
- IC5 pad 9: (no net) -> Net-(IC5-Pad9)
- J1 pad 1: USART3_TX -> Net-(J1-Pad1)
- J1 pad 2: USART3_RX -> Net-(J1-Pad2)
- J6 pad 10: (no net) -> Net-(J6-Pad10)
- J6 pad 11: (no net) -> Net-(J6-Pad11)
- J6 pad 4: (no net) -> Net-(J6-Pad4)
- J6 pad 6: (no net) -> Net-(J6-Pad6)
- J6 pad 7: (no net) -> Net-(J6-Pad7)
- J6 pad 8: (no net) -> Net-(J6-Pad8)
- J6 pad 9: (no net) -> Net-(J6-Pad9)
- Q2 pad 3: WIFI_nRST -> 3V3
- R20 pad 1: WIFI_nRST -> 3V3
- R7 pad 2: /WiFi + MCU/GPIO16 -> Net-(D4-Pad2)
- R8 pad 1: Net-(D4-Pad1) -> /WiFi + MCU/GPIO16
- R9 pad 1: WIFI_nRST -> 3V3
- SWD1 pad 2: SWCLK -> Net-(R26-Pad1)
- SWD1 pad 6: (no net) -> Net-(SWD1-Pad6)
- U1 pad 10: (no net) -> Net-(U1-Pad10)
- U1 pad 100: (no net) -> Net-(U1-Pad100)
- U1 pad 103: (no net) -> Net-(U1-Pad103)
- U1 pad 104: (no net) -> Net-(U1-Pad104)
- U1 pad 11: (no net) -> Net-(U1-Pad11)
- U1 pad 110: (no net) -> Net-(U1-Pad110)
- U1 pad 111: (no net) -> Net-(U1-Pad111)
- U1 pad 112: (no net) -> Net-(U1-Pad112)
- U1 pad 113: (no net) -> Net-(U1-Pad113)
- U1 pad 114: (no net) -> Net-(U1-Pad114)
- U1 pad 115: (no net) -> Net-(U1-Pad115)
- U1 pad 116: (no net) -> Net-(U1-Pad116)
- U1 pad 117: (no net) -> Net-(U1-Pad117)
- U1 pad 118: (no net) -> Net-(U1-Pad118)
- U1 pad 119: (no net) -> Net-(U1-Pad119)
- U1 pad 12: (no net) -> Net-(U1-Pad12)
- U1 pad 122: (no net) -> Net-(U1-Pad122)
- U1 pad 123: (no net) -> Net-(U1-Pad123)
- U1 pad 124: (no net) -> Net-(U1-Pad124)
- U1 pad 125: (no net) -> Net-(U1-Pad125)
- U1 pad 126: (no net) -> Net-(U1-Pad126)
- U1 pad 127: (no net) -> Net-(U1-Pad127)
- U1 pad 128: (no net) -> Net-(U1-Pad128)
- U1 pad 129: (no net) -> Net-(U1-Pad129)
- U1 pad 13: (no net) -> Net-(U1-Pad13)
- U1 pad 132: (no net) -> Net-(U1-Pad132)
- U1 pad 133: (no net) -> Net-(U1-Pad133)
- U1 pad 136: (no net) -> Net-(U1-Pad136)
- U1 pad 137: (no net) -> Net-(U1-Pad137)
- U1 pad 14: (no net) -> Net-(U1-Pad14)
- U1 pad 141: (no net) -> Net-(U1-Pad141)
- U1 pad 142: (no net) -> Net-(U1-Pad142)
- U1 pad 143: (no net) -> 3V3
- U1 pad 18: (no net) -> Net-(U1-Pad18)
- U1 pad 20: (no net) -> Net-(U1-Pad20)
- U1 pad 21: (no net) -> Net-(U1-Pad21)
- U1 pad 22: (no net) -> Net-(U1-Pad22)
- U1 pad 26: (no net) -> Net-(U1-Pad26)
- U1 pad 27: (no net) -> Net-(U1-Pad27)
- U1 pad 28: (no net) -> Net-(U1-Pad28)
- U1 pad 29: (no net) -> Net-(U1-Pad29)
- U1 pad 34: (no net) -> Net-(U1-Pad34)
- U1 pad 35: (no net) -> Net-(U1-Pad35)
- U1 pad 36: (no net) -> ADC123_IN2
- U1 pad 41: (no net) -> DAC_OUT2
- U1 pad 42: WIFI_nRST -> 3V3
- U1 pad 43: (no net) -> Net-(U1-Pad43)
- U1 pad 44: (no net) -> Net-(U1-Pad44)
- U1 pad 46: (no net) -> Net-(U1-Pad46)
- U1 pad 47: (no net) -> Net-(U1-Pad47)
- U1 pad 48: (no net) -> TIM2_CH4
- U1 pad 49: (no net) -> Net-(U1-Pad49)
- U1 pad 50: (no net) -> Net-(U1-Pad50)
- U1 pad 53: (no net) -> Net-(U1-Pad53)
- U1 pad 54: (no net) -> Net-(U1-Pad54)
- U1 pad 55: (no net) -> Net-(U1-Pad55)
- U1 pad 56: (no net) -> Net-(U1-Pad56)
- U1 pad 57: (no net) -> Net-(U1-Pad57)
- U1 pad 60: (no net) -> Net-(U1-Pad60)
- U1 pad 63: (no net) -> Net-(U1-Pad63)
- U1 pad 64: (no net) -> Net-(U1-Pad64)
- U1 pad 65: (no net) -> Net-(U1-Pad65)
- U1 pad 66: (no net) -> Net-(U1-Pad66)
- U1 pad 67: (no net) -> Net-(U1-Pad67)
- U1 pad 68: (no net) -> Net-(U1-Pad68)
- U1 pad 7: (no net) -> Net-(U1-Pad7)
- U1 pad 70: (no net) -> Net-(U1-Pad70)
- U1 pad 73: (no net) -> SPARE_7
- U1 pad 74: (no net) -> SPARE_6
- U1 pad 75: (no net) -> SPARE_5
- U1 pad 76: (no net) -> SPARE_4
- U1 pad 77: (no net) -> SPARE_3
- U1 pad 78: (no net) -> SPARE_2
- U1 pad 79: (no net) -> SPARE_1
- U1 pad 8: (no net) -> Net-(U1-Pad8)
- U1 pad 80: (no net) -> Net-(U1-Pad80)
- U1 pad 81: (no net) -> Net-(U1-Pad81)
- U1 pad 82: (no net) -> Net-(U1-Pad82)
- U1 pad 85: (no net) -> TIM4_CH3
- U1 pad 86: (no net) -> TIM4_CH4
- U1 pad 87: (no net) -> Net-(U1-Pad87)
- U1 pad 88: (no net) -> Net-(U1-Pad88)
- U1 pad 89: (no net) -> Net-(U1-Pad89)
- U1 pad 9: (no net) -> Net-(U1-Pad9)
- U1 pad 90: (no net) -> Net-(U1-Pad90)
- U1 pad 91: (no net) -> Net-(U1-Pad91)
- U1 pad 92: (no net) -> Net-(U1-Pad92)
- U1 pad 93: (no net) -> Net-(U1-Pad93)
- U1 pad 95: (no net) -> 3V3
- U1 pad 96: (no net) -> Net-(U1-Pad96)
- U1 pad 97: (no net) -> Net-(U1-Pad97)
- U1 pad 98: (no net) -> TIM3_CH3
- U1 pad 99: (no net) -> TIM3_CH4
- U3 pad 10: (no net) -> Net-(U3-Pad10)
- U3 pad 11: (no net) -> Net-(U3-Pad11)
- U3 pad 12: (no net) -> Net-(U3-Pad12)
- U3 pad 15: (no net) -> Net-(U3-Pad15)
- U3 pad 4: (no net) -> Net-(U3-Pad4)
- U3 pad 9: (no net) -> Net-(U3-Pad9)
Routing:
- net 3V3: track 289.9 -> 459.8 mm, vias 16 -> 22
- net WIFI_nRST: track 89.4 -> 0.00 mm, vias 3 -> 0
- net NRST: track 38.5 -> 66.3 mm
- net 5V: track 83.6 -> 67.0 mm
- net 7.5V: track 14.8 -> 28.9 mm
- net USART3_RX: track 40.3 -> 32.0 mm
- net ADC3_IN5: track 39.0 -> 47.2 mm, vias 2 -> 3
- net USART3_TX: track 43.0 -> 35.2 mm
- net Net-(J1-Pad1): track 0.00 -> 7.81 mm
- net SWCLK: track 19.2 -> 13.0 mm
- net Net-(J1-Pad2): track 0.00 -> 5.82 mm
- net Net-(R26-Pad1): track 0.00 -> 5.40 mm
- net SPARE_3: track 0.00 -> 4.70 mm, vias 0 -> 1
- net Net-(D4-Pad1): track 4.58 -> 0.00 mm
- net SPARE_5: track 0.00 -> 4.43 mm, vias 0 -> 1
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- added copper zone on B.Cu, net 5V
- removed copper zone on F.Cu, net 5V
Other:
- board text added: "Sara Hui Mohamed Ibrahim Justin Zhang Michel Raskin ECE 477 Team 7"
