File: MCU_PCB/main_controller/main_controller.kicad_pcb (KiCad board)
At the start: 2 copper layers, 94.8 x 89.5 mm, 94 parts, among them IC5 esp-12f, J1 TB006-508-05BE, J2 TB006-508-05BE, J3 VX7803-500, J4 TB006-508-05BE, J5 1715250000, J6 2174507-2, Q2 S8050, Q3 S8050, SW1 SW_SPDT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

Commit message: Finishing up small airwires
Routing:
- net 3V3: track 459.8 -> 434.6 mm
- net /WiFi + MCU/GPIO16: track 8.49 -> 12.1 mm
- net Net-(D4-Pad2): track 0.00 -> 2.96 mm
- net GND: track 35.9 -> 37.0 mm, vias 19 -> 21
