File: MCU_PCB/main_controller/file616037F9.sch (KiCad schematic (older format))
At the start: 30 parts, among them IC5 esp-12f, J8 USB_B_Micro, Q2 S8050, Q3 S8050, SW2 KEY_USER, SW3 KEY_FLASH, U3 CH340G, U4 R-78E5.0-0.5, U5 ISE0512A-H, X1 ECS-2520MV-xxx-xx

Commit message: Finalizing zipped main controller file
Parts:
- removed J8: USB_B_Micro, usbtomicro:J_SMD_2174507-2-5_7.8_5_2.71, symbol Connector:USB_B_Micro
- removed U5: ISE0512A-H, 5to3.3:ISE0512A-H, symbol 5to3.3:ISE0512A-H
- added J3: VX7803-500, walle_library:VX7803-500, symbol 5to3v3:VX7803-500
- added J6: 2174507-2, walle_library:2174507-2, symbol microusb_b:2174507-2
- D3: footprint Diode 4007:1N4007G-T -> walle_library:1N4007G-T
- IC5: footprint esp12f -> walle_library:esp12f
- SW2, SW3: footprint pushbutton:SW_147873-2 -> walle_library:SW_147873-2
- U4: footprint DC 7.5 to 5:R-78E5.0-0.5 -> walle_library:R-78E5.0-0.5
Connections:
- net labels removed: ADC
- wire segments 68 -> 64
Other:
- moved on the sheet: C23, C24, ESD1, Q2, Q3, R11, R12, R13, R14, U3

Commit message: Finally rescued footprints within the zip file - uploading to website now
Parts:
- J3: symbol 5to3v3:VX7803-500 -> main_controller-rescue:VX7803-500-5to3v3
- J6: symbol microusb_b:2174507-2 -> main_controller-rescue:2174507-2-microusb_b
- U4: symbol 7.5to5:R-78E5.0-0.5 -> main_controller-rescue:R-78E5.0-0.5-7.5to5
Changed lines of the file:
@@
 $EndComp
 $Comp
-L 7.5to5:R-78E5.0-0.5 U?
+L main_controller-rescue:R-78E5.0-0.5-7.5to5 U?
 U 1 1 615F56E0
 P 5550 3850
@@
 $EndComp
 $Comp
-L 5to3v3:VX7803-500 J3
+L main_controller-rescue:VX7803-500-5to3v3 J3
 U 1 1 6198DC88
 P 3850 3500
@@
 GND
 $Comp
-L microusb_b:2174507-2 J6
+L main_controller-rescue:2174507-2-microusb_b J6
 U 1 1 6199C811
 P 9750 5350

Commit message: mounting holes and test points
Parts:
- added H1, H2, H3: MountingHole, MountingHole:MountingHole_2.2mm_M2, symbol Mechanical:MountingHole
- added TP1, TP2: TestPoint, TestPoint:TestPoint_Loop_D2.50mm_Drill1.0mm, symbol Connector:TestPoint
- J3: symbol main_controller-rescue:VX7803-500-5to3v3 -> 5to3v3:VX7803-500
- J6: symbol main_controller-rescue:2174507-2-microusb_b -> microusb_b:2174507-2
- U4: symbol main_controller-rescue:R-78E5.0-0.5-7.5to5 -> 7.5to5:R-78E5.0-0.5
Changed lines of the file:
@@
 $EndComp
 $Comp
-L main_controller-rescue:R-78E5.0-0.5-7.5to5 U?
+L 7.5to5:R-78E5.0-0.5 U?
 U 1 1 615F56E0
 P 5550 3850
@@
 $EndComp
 $Comp
-L main_controller-rescue:VX7803-500-5to3v3 J3
+L 5to3v3:VX7803-500 J3
 U 1 1 6198DC88
 P 3850 3500
@@
 GND
 $Comp
-L main_controller-rescue:2174507-2-microusb_b J6
+L microusb_b:2174507-2 J6
 U 1 1 6199C811
 P 9750 5350
@@
 Text GLabel 9750 5750 0    39   Input ~ 0
 GND
+$Comp
+L Connector:TestPoint TP1
+U 1 1 61A9A436
+P 2300 2850
+F 0 "TP1" H 2358 2968 50  0000 L CNN
+F 1 "TestPoint" H 2358 2877 50  0000 L CNN
+F 2 "TestPoint:TestPoint_Loop_D2.50mm_Drill1.0mm" H 2500 2850 50  0001 C CNN
+F 3 "~" H 2500 2850 50  0001 C CNN
+	1    2300 2850
+	1    0    0    -1
+$EndComp
+Text GLabel 2300 2850 3    39   Input ~ 0
+USART1_TX
+$Comp
+L Connector:TestPoint TP2
+U 1 1 61A9BF95
+P 2950 2850
+F 0 "TP2" H 3008 2968 50  0000 L CNN
+F 1 "TestPoint" H 3008 2877 50  0000 L CNN
+F 2 "TestPoint:TestPoint_Loop_D2.50mm_Drill1.0mm" H 3150 2850 50  0001 C CNN
+F 3 "~" H 3150 2850 50  0001 C CNN
+	1    2950 2850
+	1    0    0    -1
+$EndComp
+Text GLabel 2950 2850 3    39   Input ~ 0
+USART1_RX
+$Comp
+L Mechanical:MountingHole H1
+U 1 1 61A9F739
+P 6200 2600
+F 0 "H1" H 6300 2646 50  0000 L CNN
+F 1 "MountingHole" H 6300 2555 50  0000 L CNN
+F 2 "MountingHole:MountingHole_2.2mm_M2" H 6200 2600 50  0001 C CNN
+F 3 "~" H 6200 2600 50  0001 C CNN
+	1    6200 2600
+	1    0    0    -1
+$EndComp
+$Comp
+L Mechanical:MountingHole H2
+U 1 1 61AA5D09
+P 6200 2900
+F 0 "H2" H 6300 2946 50  0000 L CNN
+F 1 "MountingHole" H 6300 2855 50  0000 L CNN
+F 2 "MountingHole:MountingHole_2.2mm_M2" H 6200 2900 50  0001 C CNN
+F 3 "~" H 6200 2900 50  0001 C CNN
+	1    6200 2900
+	1    0    0    -1
+$EndComp
+$Comp
+L Mechanical:MountingHole H3
+U 1 1 61AA7533
+P 6200 3200
+F 0 "H3" H 6300 3246 50  0000 L CNN
+F 1 "MountingHole" H 6300 3155 50  0000 L CNN
+F 2 "MountingHole:MountingHole_2.2mm_M2" H 6200 3200 50  0001 C CNN
+F 3 "~" H 6200 3200 50  0001 C CNN
+	1    6200 3200
+	1    0    0    -1
+$EndComp
 $EndSCHEMATC

Commit message: Increasing 5V Trace
Connections:
- wire segments 64 -> 67
Other:
- moved on the sheet: Q2
Changed lines of the file:
@@
 nRST
-Wire Wire Line
-	1100 5100 1100 4750
 Wire Wire Line
 	1100 6450 1100 7050
@@
 	1    2350 5300
 	0    1    1    0
-$EndComp
-$Comp
-L Transistor_BJT:S8050 Q3
-U 1 1 6155F7AE
-P 1200 6250
-F 0 "Q3" H 1391 6204 50  0000 L CNN
-F 1 "S8050" H 1391 6295 50  0000 L CNN
-F 2 "Package_TO_SOT_THT:TO-92_Inline" H 1400 6175 50  0001 L CIN
-F 3 "http://www.unisonic.com.tw/datasheet/S8050.pdf" H 1200 6250 50  0001 L CNN
-	1    1200 6250
-	-1   0    0    1
-$EndComp
-$Comp
-L Transistor_BJT:S8050 Q2
-U 1 1 61561FA1
-P 1200 5300
-F 0 "Q2" H 1391 5254 50  0000 L CNN
-F 1 "S8050" H 1391 5345 50  0000 L CNN
-F 2 "Package_TO_SOT_THT:TO-92_Inline" H 1400 5225 50  0001 L CIN
-F 3 "http://www.unisonic.com.tw/datasheet/S8050.pdf" H 1200 5300 50  0001 L CNN
-	1    1200 5300
-	-1   0    0    1
 $EndComp
 $Comp
@@
 	1    0    0    -1
 $EndComp
+$Comp
+L Transistor_BJT:S8050 Q2
+U 1 1 61561FA1
+P 1000 5300
+F 0 "Q2" H 1191 5254 50  0000 L CNN
+F 1 "S8050" H 1191 5345 50  0000 L CNN
+F 2 "Package_TO_SOT_THT:TO-92_Inline" H 1200 5225 50  0001 L CIN
+F 3 "http://www.unisonic.com.tw/datasheet/S8050.pdf" H 1000 5300 50  0001 L CNN
+	1    1000 5300
+	1    0    0    -1
+$EndComp
+Wire Wire Line
+	1100 5100 1100 4750
+Wire Wire Line
+	1400 5300 1400 5600
+Wire Wire Line
+	1400 5600 800  5600
+Wire Wire Line
+	800  5600 800  5300
+$Comp
+L Transistor_BJT:S8050 Q3
+U 1 1 6155F7AE
+P 1200 6250
+F 0 "Q3" H 1391 6204 50  0000 L CNN
+F 1 "S8050" H 1391 6295 50  0000 L CNN
+F 2 "Package_TO_SOT_THT:TO-92_Inline" H 1400 6175 50  0001 L CIN
+F 3 "http://www.unisonic.com.tw/datasheet/S8050.pdf" H 1200 6250 50  0001 L CNN
+	1    1200 6250
+	-1   0    0    1
+$EndComp
 $EndSCHEMATC

Commit message: Final
Parts:
- removed U4: R-78E5.0-0.5, walle_library:R-78E5.0-0.5, symbol 7.5to5:R-78E5.0-0.5
- added C22, C28, C29: 10uF, Capacitor_SMD:C_1210_3225Metric, symbol Device:C
- added C27: 22uF, Capacitor_SMD:C_1210_3225Metric, symbol Device:C
- added PS1: R-78E5.0-1.0, R78E5010, symbol R-78E5.0-1.0:R-78E5.0-1.0
- J3: symbol 5to3v3:VX7803-500 -> main_controller-rescue:VX7803-500-5to3v3
- J6: symbol microusb_b:2174507-2 -> main_controller-rescue:2174507-2-microusb_b
Connections:
- wire segments 67 -> 75
Changed lines of the file:
@@
 	1    0    0    -1
 $EndComp
-Text GLabel 5550 3850 0    50   Input ~ 0
+Text GLabel 5300 3800 0    50   Input ~ 0
 7.5V
-Text GLabel 7150 3850 2    50   Input ~ 0
+Text GLabel 5300 4000 0    50   Input ~ 0
 5V
-Text GLabel 7150 3950 2    50   Input ~ 0
+Text GLabel 5750 3900 0    50   Input ~ 0
 GND
 Text GLabel 5600 5450 0    25   Input ~ 0
@@
 	2650 5300 4050 5300
 Connection ~ 2650 5300
-Wire Wire Line
-	3000 5250 4050 5250
 Text Label 1100 7050 0    50   ~ 0
 GPIO0
@@
 	1100 6050 2650 6050
 Wire Wire Line
-	2750 6250 3000 6250
-Connection ~ 2750 6250
-Wire Wire Line
-	2750 5500 2750 6250
-Wire Wire Line
 	1100 5500 2750 5500
 Wire Wire Line
@@
 Wire Wire Line
 	3000 6250 3000 5250
-Wire Wire Line
-	2500 6250 2750 6250
 Wire Wire Line
 	1400 6250 2200 6250
@@
 $EndComp
 $Comp
-L 7.5to5:R-78E5.0-0.5 U?
-U 1 1 615F56E0
-P 5550 3850
-AR Path="/61651051/615F56E0" Ref="U?"  Part="1"
-AR Path="/616037FA/615F56E0" Ref="U4"  Part="1"
-F 0 "U4" H 6350 4237 60  0000 C CNN
-F 1 "R-78E5.0-0.5" H 6350 4131 60  0000 C CNN
-F 2 "walle_library:R-78E5.0-0.5" H 6350 4090 60  0001 C CNN
-F 3 "" H 5550 3850 60  0000 C CNN
-	1    5550 3850
-	1    0    0    -1
-$EndComp
-$Comp
-L 5to3v3:VX7803-500 J3
+L main_controller-rescue:VX7803-500-5to3v3 J3
 U 1 1 6198DC88
 P 3850 3500
+AR Path="/6198DC88" Ref="J3"  Part="1"
+AR Path="/616037FA/6198DC88" Ref="J3"  Part="1"
 F 0 "J3" H 4378 3453 60  0000 L CNN
 F 1 "VX7803-500" H 4378 3347 60  0000 L CNN
@@
 	1    0    0    -1
 $EndComp
-Text GLabel 3850 3500 0    39   Input ~ 0
+Text GLabel 3350 3500 0    39   Input ~ 0
 5V
-Text GLabel 3850 3700 0    39   Input ~ 0
+Text GLabel 3400 3700 0    39   Input ~ 0
 3V3
 Text GLabel 3850 3600 0    39   Input ~ 0
 GND
 $Comp
-L microusb_b:2174507-2 J6
+L main_controller-rescue:2174507-2-microusb_b J6
 U 1 1 6199C811
 P 9750 5350
@@
 $EndComp
 Wire Wire Line
-	1100 5100 1100 4750
-Wire Wire Line
 	1400 5300 1400 5600
 Wire Wire Line
 	1400 5600 800  5600
-Wire Wire Line
-	800  5600 800  5300
 $Comp
 L Transistor_BJT:S8050 Q3
@@
 	-1   0    0    1
 $EndComp
+$Comp
+L Device:C C22
+U 1 1 6171223D
+P 3650 3350
+F 0 "C22" H 3765 3396 50  0000 L CNN
+F 1 "10uF" H 3765 3305 50  0000 L CNN
+F 2 "Capacitor_SMD:C_1210_3225Metric" H 3688 3200 50  0001 C CNN
+F 3 "~" H 3650 3350 50  0001 C CNN
+	1    3650 3350
+	1    0    0    -1
+$EndComp
+Wire Wire Line
+	3350 3500 3650 3500
+Connection ~ 3650 3500
+Wire Wire Line
+	3650 3500 3850 3500
+Text GLabel 3650 3200 0    50   Input ~ 0
+GND
+$Comp
+L Device:C C27
+U 1 1 61719C85
+P 3650 3850
+F 0 "C27" H 3765 3896 50  0000 L CNN
+F 1 "22uF" H 3765 3805 50  0000 L CNN
+F 2 "Capacitor_SMD:C_1210_3225Metric" H 3688 3700 50  0001 C CNN
+F 3 "~" H 3650 3850 50  0001 C CNN
+	1    3650 3850
+	1    0    0    -1
+$EndComp
+Wire Wire Line
+	3400 3700 3650 3700
+Connection ~ 3650 3700
+Wire Wire Line
+	3650 3700 3850 3700
+Text GLabel 3650 4000 0    50   Input ~ 0
+GND
+$Comp
+L R-78E5.0-1.0:R-78E5.0-1.0 PS1
+U 1 1 6171FA76
+P 5750 3800
+F 0 "PS1" H 6578 3746 50  0000 L CNN
+F 1 "R-78E5.0-1.0" H 6578 3655 50  0000 L CNN
+F 2 "R78E5010" H 6600 3900 50  0001 L CNN
+F 3 "http://www.recom-power.com/pdf/Innoline/R-78Exx-1.0.pdf" H 6600 3800 50  0001 L CNN
+F 4 "Non-Isolated DC/DC Converters 8-28Vin 5V 1.0A THRU" H 6600 3700 50  0001 L CNN "Description"
+F 5 "10.4" H 6600 3600 50  0001 L CNN "Height"
+F 6 "919-R-78E5.0-1.0" H 6600 3500 50  0001 L CNN "Mouser Part Number"
+F 7 "https://www.mouser.co.uk/ProductDetail/RECOM-Power/R-78E50-10?qs=T0XSgvH75d4EsZCU9I5HVA%3D%3D" H 6600 3400 50  0001 L CNN "Mouser Price/Stock"
+F 8 "RECOM Power" H 6600 3300 50  0001 L CNN "Manufacturer_Name"
+F 9 "R-78E5.0-1.0" H 6600 3200 50  0001 L CNN "Manufacturer_Part_Number"
+	1    5750 3800
+	1    0    0    -1
+$EndComp
+$Comp
+L Device:C C28
+U 1 1 61725B78
+P 5500 3650
+F 0 "C28" H 5615 3696 50  0000 L CNN
+F 1 "10uF" H 5615 3605 50  0000 L CNN
+F 2 "Capacitor_SMD:C_1210_3225Metric" H 5538 3500 50  0001 C CNN
+F 3 "~" H 5500 3650 50  0001 C CNN
+	1    5500 3650
+	1    0    0    -1
+$EndComp
+$Comp
+L Device:C C29
+U 1 1 617277D0
+P 5500 4150
+F 0 "C29" H 5615 4196 50  0000 L CNN
+F 1 "10uF" H 5615 4105 50  0000 L CNN
+F 2 "Capacitor_SMD:C_1210_3225Metric" H 5538 4000 50  0001 C CNN
+F 3 "~" H 5500 4150 50  0001 C CNN
+	1    5500 4150
+	1    0    0    -1
+$EndComp
+Wire Wire Line
+	5300 4000 5500 4000
+Connection ~ 5500 4000
+Wire Wire Line
+	5500 4000 5750 4000
+Wire Wire Line
+	5300 3800 5500 3800
+Connection ~ 5500 3800
+Wire Wire Line
+	5500 3800 5750 3800
+Text GLabel 5500 3500 0    50   Input ~ 0
+GND
+Text GLabel 5500 4300 0    50   Input ~ 0
+GND
+Wire Wire Line
+	1100 5100 1100 4750
+Wire Wire Line
+	800  5600 800  5300
+Wire Wire Line
+	4050 5250 3000 5250
+Wire Wire Line
+	3000 6250 2750 6250
+Wire Wire Line
+	2750 5500 2750 6250
+Connection ~ 2750 6250
+Wire Wire Line
+	2750 6250 2500 6250
 $EndSCHEMATC

Commit message: Almost approved
Parts:
- removed X1: ECS-2520MV-xxx-xx, Oscillator:Oscillator_SMD_ECS_2520MV-xxx-xx-4Pin_2.5x2.0mm, symbol Oscillator:ECS-2520MV-xxx-xx
- added Y2: ABM3B-12.000MHZ, walle_library:ABM3B-12.000MHZ, symbol 2021-10-20_16-14-19:ABM3B-12.000MHZ
- C18: footprint EEEHA0J101WR:CAP_EEEHA0J101WR -> walle_library:CAP_EEEHA0J101WR
- TP1, TP2: footprint TestPoint:TestPoint_Loop_D2.50mm_Drill1.0mm -> walle_library:KEYSTONE_5000
Connections:
- net WIFI_nRST is gone; now on net 3V3: C19.2, IC5.1 (RST), Q2.3 (C), R20.1, R9.1
- net GND: now also Y2.2 (GND), Y2.4 (GND)
- net GPIO16: now also D4.1 (K), R8.1; no longer D4.2 (A), R7.2
- net XI: now also Y2.3 (2)
- net XO: now also Y2.1
- new net: D4.2 (A), R7.2
Other:
- moved on the sheet: C25, C26
Changed lines of the file:
@@
 Text Label 8850 2800 0    50   ~ 0
 3V3
-Wire Wire Line
-	8850 3550 8850 3650
 $Comp
 L Device:R R8
@@
 $EndComp
 Wire Wire Line
-	8850 4000 8850 4200
+	8850 4000 8850 4100
 $Comp
 L Switch:SW_Push SW2
@@
 $EndComp
 Wire Wire Line
-	8850 3650 8550 3650
-Connection ~ 8850 3650
-Wire Wire Line
-	8850 3650 8850 3700
-Text Label 8550 3650 2    50   ~ 0
+	8850 4100 8550 4100
+Text Label 8550 4100 2    50   ~ 0
 GPIO16
 Wire Wire Line
@@
 F 0 "C18" H 4865 2096 50  0000 L CNN
 F 1 "100uF" H 4865 2005 50  0000 L CNN
-F 2 "EEEHA0J101WR:CAP_EEEHA0J101WR" H 4750 2050 50  0001 C CNN
+F 2 "walle_library:CAP_EEEHA0J101WR" H 4750 2050 50  0001 C CNN
 F 3 "~" H 4750 2050 50  0001 C CNN
 	1    4750 2050
@@
 Wire Wire Line
 	3900 6650 4350 6650
-$Comp
-L Oscillator:ECS-2520MV-xxx-xx X1
-U 1 1 615543D8
-P 9500 1250
-F 0 "X1" H 9944 1296 50  0000 L CNN
-F 1 "ECS-2520MV-xxx-xx" H 9944 1205 50  0000 L CNN
-F 2 "Oscillator:Oscillator_SMD_ECS_2520MV-xxx-xx-4Pin_2.5x2.0mm" H 9950 900 50  0001 C CNN
-F 3 "https://www.ecsxtal.com/store/pdf/ECS-2520MV.pdf" H 9325 1375 50  0001 C CNN
-	1    9500 1250
-	1    0    0    -1
-$EndComp
-Wire Wire Line
-	9100 1250 8800 1250
-Wire Wire Line
-	8800 1250 8800 1450
-Text Label 8800 1750 3    50   ~ 0
-GND
-Wire Wire Line
-	9900 1250 9900 1450
-Wire Wire Line
-	9900 1450 10150 1450
-Text Label 10150 1750 3    50   ~ 0
+Text Label 8850 1600 3    50   ~ 0
+GND
+Text Label 9650 1600 3    50   ~ 0
 GND
 $Comp
 L Device:C C26
 U 1 1 615557B3
-P 10150 1600
-F 0 "C26" H 10265 1691 50  0000 L CNN
-F 1 "22pF" H 10265 1600 50  0000 L CNN
-F 2 "Capacitor_SMD:C_0805_2012Metric" H 10265 1509 50  0000 L CNN
-F 3 "~" H 10150 1600 50  0001 C CNN
-	1    10150 1600
-	1    0    0    -1
-$EndComp
-Text Label 9500 1550 3    50   ~ 0
-GND
-Text Label 9500 950  0    50   ~ 0
-GND
-Text Label 8800 1250 2    50   ~ 0
-XO
+P 9650 1450
+F 0 "C26" H 9765 1541 50  0000 L CNN
+F 1 "22pF" H 9765 1450 50  0000 L CNN
+F 2 "Capacitor_SMD:C_0805_2012Metric" H 9765 1359 50  0000 L CNN
+F 3 "~" H 9650 1450 50  0001 C CNN
+	1    9650 1450
+	1    0    0    -1
+$EndComp
 Text Label 9100 4900 3    50   ~ 0
 GND
@@
 L Device:C C25
 U 1 1 61555339
-P 8800 1600
-F 0 "C25" H 8915 1691 50  0000 L CNN
-F 1 "22pF" H 8915 1600 50  0000 L CNN
-F 2 "Capacitor_SMD:C_0805_2012Metric" H 8915 1509 50  0000 L CNN
-F 3 "~" H 8800 1600 50  0001 C CNN
-	1    8800 1600
+P 8850 1450
+F 0 "C25" H 8965 1541 50  0000 L CNN
+F 1 "22pF" H 8965 1450 50  0000 L CNN
+F 2 "Capacitor_SMD:C_0805_2012Metric" H 8965 1359 50  0000 L CNN
+F 3 "~" H 8850 1450 50  0001 C CNN
+	1    8850 1450
 	1    0    0    -1
 $EndComp
@@
 Text GLabel 4850 5750 2    25   Input ~ 0
 USB_D+
-Text Label 10050 1450 0    50   ~ 0
-XI
 Wire Wire Line
 	3450 5950 3400 5950
@@
 F 0 "TP1" H 2358 2968 50  0000 L CNN
 F 1 "TestPoint" H 2358 2877 50  0000 L CNN
-F 2 "TestPoint:TestPoint_Loop_D2.50mm_Drill1.0mm" H 2500 2850 50  0001 C CNN
+F 2 "walle_library:KEYSTONE_5000" H 2500 2850 50  0001 C CNN
 F 3 "~" H 2500 2850 50  0001 C CNN
 	1    2300 2850
@@
 F 0 "TP2" H 3008 2968 50  0000 L CNN
 F 1 "TestPoint" H 3008 2877 50  0000 L CNN
-F 2 "TestPoint:TestPoint_Loop_D2.50mm_Drill1.0mm" H 3150 2850 50  0001 C CNN
+F 2 "walle_library:KEYSTONE_5000" H 3150 2850 50  0001 C CNN
 F 3 "~" H 3150 2850 50  0001 C CNN
 	1    2950 2850
@@
 Wire Wire Line
 	2750 6250 2500 6250
+Connection ~ 8850 4100
+Wire Wire Line
+	8850 4100 8850 4200
+Wire Wire Line
+	8850 3550 8850 3700
+Wire Wire Line
+	9400 4000 9400 3750
+Connection ~ 9400 4000
+Text Label 9400 3750 0    50   ~ 0
+3V3
+$Comp
+L 2021-10-20_16-14-19:ABM3B-12.000MHZ Y2
+U 1 1 61811995
+P 8950 1300
+F 0 "Y2" H 9394 1353 60  0000 L CNN
+F 1 "ABM3B-12.000MHZ" H 9394 1247 60  0000 L CNN
+F 2 "walle_library:ABM3B-12.000MHZ" H 9150 940 60  0001 C CNN
+F 3 "" H 8950 1300 60  0000 C CNN
+	1    8950 1300
+	1    0    0    -1
+$EndComp
+Wire Wire Line
+	8850 1300 8950 1300
+Wire Wire Line
+	9350 1300 9650 1300
+Text Label 8850 1300 2    50   ~ 0
+XO
+Text Label 9650 1300 0    50   ~ 0
+XI
+Text Label 9150 1100 0    50   ~ 0
+GND
+Text Label 9150 1500 3    50   ~ 0
+GND
 $EndSCHEMATC

Commit message: Finishing up small airwires
Parts:
- C18: symbol Device:CP1 -> main_controller-rescue:CP1-Device
- C19, C22, C23, C24, C25, C26, C27, C28, C29: symbol Device:C -> main_controller-rescue:C-Device
- D3: symbol Device:D_Schottky -> main_controller-rescue:D_Schottky-Device
- D4: symbol Device:LED -> main_controller-rescue:LED-Device
- H1, H2, H3: symbol Mechanical:MountingHole -> main_controller-rescue:MountingHole-Mechanical
- PS1: symbol R-78E5.0-1.0:R-78E5.0-1.0 -> main_controller-rescue:R-78E5.0-1.0-R-78E5.0-1.0
- Q2, Q3: symbol Transistor_BJT:S8050 -> main_controller-rescue:S8050-Transistor_BJT
- R10, R11, R12, R13, R14, R17, R19, R20, R7, R8, R9: symbol Device:R -> main_controller-rescue:R-Device
- SW2, SW3: symbol Switch:SW_Push -> main_controller-rescue:SW_Push-Switch
- TP1, TP2: symbol Connector:TestPoint -> main_controller-rescue:TestPoint-Connector
- U3: symbol Interface_USB:CH340G -> main_controller-rescue:CH340G-Interface_USB
- Y2: symbol 2021-10-20_16-14-19:ABM3B-12.000MHZ -> main_controller-rescue:ABM3B-12.000MHZ-2021-10-20_16-14-19
Changed lines of the file:
@@
 NoConn ~ 4850 5950
 $Comp
-L Device:C C24
+L main_controller-rescue:C-Device C24
 U 1 1 6156B43A
 P 4350 6800
@@
 $EndComp
 $Comp
-L Device:C C23
+L main_controller-rescue:C-Device C23
 U 1 1 6156C5A8
 P 3900 6800
@@
 GND
 $Comp
-L power:GND #PWR0126
+L main_controller-rescue:GND-power #PWR0126
 U 1 1 615791C3
 P 10950 6250
@@
 GND
 $Comp
-L Device:R R7
+L main_controller-rescue:R-Device R7
 U 1 1 615DD82A
 P 8850 3400
@@
 $EndComp
 $Comp
-L Device:LED D4
+L main_controller-rescue:LED-Device D4
 U 1 1 615DE183
 P 8850 3850
@@
 3V3
 $Comp
-L Device:R R8
+L main_controller-rescue:R-Device R8
 U 1 1 615E2601
 P 8850 4350
@@
 	8850 4000 8850 4100
 $Comp
-L Switch:SW_Push SW2
+L main_controller-rescue:SW_Push-Switch SW2
 U 1 1 615E55B3
 P 9100 4700
@@
 	8850 4500 9100 4500
 $Comp
-L Device:R R9
+L main_controller-rescue:R-Device R9
 U 1 1 615EA1F0
 P 9400 4350
@@
 nRST
 $Comp
-L Device:R R10
+L main_controller-rescue:R-Device R10
 U 1 1 615F113F
 P 10500 4300
@@
 $EndComp
 $Comp
-L Switch:SW_Push SW3
+L main_controller-rescue:SW_Push-Switch SW3
 U 1 1 615F1B1E
 P 10500 4650
@@
 3V3
 $Comp
-L Device:CP1 C18
+L main_controller-rescue:CP1-Device C18
 U 1 1 616121AA
 P 4750 2050
@@
 GND
 $Comp
-L Device:R R17
+L main_controller-rescue:R-Device R17
 U 1 1 6161B737
 P 1400 950
@@
 $EndComp
 $Comp
-L Device:R R19
+L main_controller-rescue:R-Device R19
 U 1 1 6161C48F
 P 1400 1250
@@
 $EndComp
 $Comp
-L Device:R R20
+L main_controller-rescue:R-Device R20
 U 1 1 61621E60
 P 1400 1550
@@
 	1550 1550 1800 1550
 $Comp
-L Device:C C19
+L main_controller-rescue:C-Device C19
 U 1 1 616533B8
 P 1950 1550
@@
 GND
 $Comp
-L Device:R R13
+L main_controller-rescue:R-Device R13
 U 1 1 616FEA42
 P 3600 5950
@@
 $EndComp
 $Comp
-L Device:R R14
+L main_controller-rescue:R-Device R14
 U 1 1 616FFC38
 P 3600 6250
@@
 GND
 $Comp
-L Device:C C26
+L main_controller-rescue:C-Device C26
 U 1 1 615557B3
 P 9650 1450
@@
 USART1_RX
 $Comp
-L Device:C C25
+L main_controller-rescue:C-Device C25
 U 1 1 61555339
 P 8850 1450
@@
 	6000 5150 6300 5150
 $Comp
-L power:+5V #PWR?
+L main_controller-rescue:+5V-power #PWR?
 U 1 1 616D6E25
 P 6300 5150
@@
 	6000 5950 6000 6050
 $Comp
-L power:GND #PWR?
+L main_controller-rescue:GND-power #PWR?
 U 1 1 616D6E2C
 P 6000 6050
@@
 	3450 6250 3400 6250
 $Comp
-L Interface_USB:CH340G U3
+L main_controller-rescue:CH340G-Interface_USB U3
 U 1 1 6155C867
 P 4450 5650
@@
 	1400 6250 2200 6250
 $Comp
-L Device:R R12
+L main_controller-rescue:R-Device R12
 U 1 1 61564667
 P 2350 6250
@@
 $EndComp
 $Comp
-L Device:R R11
+L main_controller-rescue:R-Device R11
 U 1 1 61563235
 P 2350 5300
@@
 $EndComp
 $Comp
-L Device:D_Schottky D3
+L main_controller-rescue:D_Schottky-Device D3
 U 1 1 619A2A55
 P 9600 5350
@@
 GND
 $Comp
-L Connector:TestPoint TP1
+L main_controller-rescue:TestPoint-Connector TP1
 U 1 1 61A9A436
 P 2300 2850
@@
 USART1_TX
 $Comp
-L Connector:TestPoint TP2
+L main_controller-rescue:TestPoint-Connector TP2
 U 1 1 61A9BF95
 P 2950 2850
@@
 USART1_RX
 $Comp
-L Mechanical:MountingHole H1
+L main_controller-rescue:MountingHole-Mechanical H1
 U 1 1 61A9F739
 P 6200 2600
@@
 $EndComp
 $Comp
-L Mechanical:MountingHole H2
+L main_controller-rescue:MountingHole-Mechanical H2
 U 1 1 61AA5D09
 P 6200 2900
@@
 $EndComp
 $Comp
-L Mechanical:MountingHole H3
+L main_controller-rescue:MountingHole-Mechanical H3
 U 1 1 61AA7533
 P 6200 3200
@@
 $EndComp
 $Comp
-L Transistor_BJT:S8050 Q2
+L main_controller-rescue:S8050-Transistor_BJT Q2
 U 1 1 61561FA1
 P 1000 5300
@@
 	1400 5600 800  5600
 $Comp
-L Transistor_BJT:S8050 Q3
+L main_controller-rescue:S8050-Transistor_BJT Q3
 U 1 1 6155F7AE
 P 1200 6250
@@
 $EndComp
 $Comp
-L Device:C C22
+L main_controller-rescue:C-Device C22
 U 1 1 6171223D
 P 3650 3350
@@
 GND
 $Comp
-L Device:C C27
+L main_controller-rescue:C-Device C27
 U 1 1 61719C85
 P 3650 3850
@@
 GND
 $Comp
-L R-78E5.0-1.0:R-78E5.0-1.0 PS1
+L main_controller-rescue:R-78E5.0-1.0-R-78E5.0-1.0 PS1
 U 1 1 6171FA76
 P 5750 3800
@@
 $EndComp
 $Comp
-L Device:C C28
+L main_controller-rescue:C-Device C28
 U 1 1 61725B78
 P 5500 3650
@@
 $EndComp
 $Comp
-L Device:C C29
+L main_controller-rescue:C-Device C29
 U 1 1 617277D0
 P 5500 4150
@@
 3V3
 $Comp
-L 2021-10-20_16-14-19:ABM3B-12.000MHZ Y2
+L main_controller-rescue:ABM3B-12.000MHZ-2021-10-20_16-14-19 Y2
 U 1 1 61811995
 P 8950 1300
+AR Path="/61811995" Ref="Y2"  Part="1"
+AR Path="/616037FA/61811995" Ref="Y2"  Part="1"
 F 0 "Y2" H 9394 1353 60  0000 L CNN
 F 1 "ABM3B-12.000MHZ" H 9394 1247 60  0000 L CNN
